File: HW/Sensor_Node.kicad_pcb (KiCad board)
At the start: 2 copper layers, 50 x 50 mm, 59 parts, among them P1 SWIM, P10 VIN, P11 IIC, P2 NTC, P3 LDR, P4 485, P5 IR, P6 LED2, P7 RADAR, P8 GAS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

Commit message: PCB Update
Parts:
- added C14: 100n, Capacitors_SMD:C_0805, F.Cu at (108.2, 83.1)
- P7: footprint Motion_Node:JST_B3B-XH-A -> Motion_Node:RCWL-0516_3Pin; moved to B.Cu
- U7: value AP1117D33 -> AMS1117
- moved C6 47.0 mm to (104.5, 90.4), turned to 180 degrees
- moved P11 44.7 mm to (103.8, 53.4)
- moved C4 44.7 mm to (92.8, 78.9)
- moved C7 44.7 mm to (92.8, 82.6)
- moved C8 44.7 mm to (107.5, 74.7)
- moved D4 44.7 mm to (114.0, 79.1)
- moved JP4 44.7 mm to (108.4, 63.2)
- moved R2 44.7 mm to (111.7, 88.1)
- moved R7 44.7 mm to (107.5, 78.2)
- moved C1 44.7 mm to (90.4, 78.9)
- moved C11 44.7 mm to (75.9, 80.6)
- moved C12 44.7 mm to (75.9, 82.5)
- moved C13 44.7 mm to (76.0, 68.3)
- moved C2 44.7 mm to (92.0, 55.1)
- moved C3 44.7 mm to (92.0, 53.2)
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Routing:
- net /NTC: track 40.0 -> 41.9 mm
- net /GAS: track 48.9 -> 47.3 mm
- net Net-(D4-Pad2): track 11.4 -> 9.90 mm
- net /RX_485: track 51.0 -> 49.7 mm
- net /TX_485: track 44.2 -> 43.2 mm
- net /RADAR: track 48.0 -> 49.0 mm
- net /DE_485: track 42.5 -> 41.5 mm
- net GND: track 100.7 -> 101.4 mm, vias 3 -> 5
- net /STATUS_3: track 29.9 -> 30.4 mm
- net Net-(P4-Pad3): track 10.3 -> 9.75 mm
