File: HW/Sensor_Node.sch (KiCad schematic (older format))
At the start: 56 parts, among them P1 SWIM, P10 VIN, P11 IIC, P2 NTC, P3 LDR, P4 485, P5 IR, P6 LED2, P7 RADAR, P8 GAS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

Commit message: PCB Update
Parts:
- removed U7: AP1117D33, TO_SOT_Packages_SMD:SOT-223, symbol AP1117D33
- added C14: 100n, Capacitors_SMD:C_0805, symbol C_Cer_SMD_0805
- added U7: AMS1117, TO_SOT_Packages_SMD:SOT-223, symbol AMS1117
- P7: footprint Motion_Node:JST_B3B-XH-A -> Motion_Node:RCWL-0516_3Pin
Connections:
- wire segments 230 -> 232
- no-connect marks 4 -> 6
Changed lines of the file:
@@
 Comment4 ""
 $EndDescr
-$Comp
-L STM8S105K4 U2
-U 1 1 5A23A0F3
-P 3150 2500
-F 0 "U2" H 1950 3500 60  0000 C CNN
-F 1 "STM8S105K4" H 4050 3500 60  0000 C CNN
-F 2 "Housings_QFP:LQFP-32_7x7mm_Pitch0.8mm" H 3200 1200 60  0001 C CNN
-F 3 "http://www.st.com/st-web-ui/static/active/en/resource/technical/document/datasheet/CD00200092.pdf" H 3100 1350 60  0001 C CNN
-	1    3150 2500
-	1    0    0    -1
-$EndComp
 Wire Wire Line
 	4500 3100 5000 3100
@@
 	1250 6050 1100 6050
 Wire Wire Line
-	1100 6050 1100 6100
-Wire Wire Line
 	1250 6250 1100 6250
 Wire Wire Line
@@
 	2400 6250 2400 6300
 $Comp
-L AP1117D33 U7
-U 1 1 5A23CCC0
-P 1350 7000
-F 0 "U7" H 1450 6750 50  0000 C CNN
-F 1 "AP1117D33" H 1350 7250 50  0000 C CNN
-F 2 "TO_SOT_Packages_SMD:SOT-223" H 1350 7000 50  0001 C CNN
-F 3 "" H 1350 7000 50  0000 C CNN
-	1    1350 7000
-	1    0    0    -1
-$EndComp
-$Comp
 L GND #PWR011
 U 1 1 5A23CDEE
-P 1350 7400
-F 0 "#PWR011" H 1350 7150 50  0001 C CNN
-F 1 "GND" H 1350 7250 50  0000 C CNN
-F 2 "" H 1350 7400 50  0000 C CNN
-F 3 "" H 1350 7400 50  0000 C CNN
-	1    1350 7400
-	1    0    0    -1
-$EndComp
-Wire Wire Line
-	1350 7300 1350 7400
-Wire Wire Line
-	1050 7000 800  7000
+P 1250 7400
+F 0 "#PWR011" H 1250 7150 50  0001 C CNN
+F 1 "GND" H 1250 7250 50  0000 C CNN
+F 2 "" H 1250 7400 50  0000 C CNN
+F 3 "" H 1250 7400 50  0000 C CNN
+	1    1250 7400
+	1    0    0    -1
+$EndComp
 Wire Wire Line
 	800  7000 800  6950
@@
 F 0 "P7" H 10850 4550 50  0000 C CNN
 F 1 "RADAR" V 10950 4350 50  0000 C CNN
-F 2 "Motion_Node:JST_B3B-XH-A" H 10850 4350 50  0001 C CNN
+F 2 "Motion_Node:RCWL-0516_3Pin" H 10850 4350 50  0001 C CNN
 F 3 "" H 10850 4350 50  0000 C CNN
 	1    10850 4350
@@
 Connection ~ 2050 7300
 Connection ~ 2325 7000
+$Comp
+L C_Cer_SMD_0805 C14
+U 1 1 5A24DC01
+P 6325 3275
+F 0 "C14" H 6335 3345 50  0000 L CNN
+F 1 "100n" H 6335 3195 50  0000 L CNN
+F 2 "Capacitors_SMD:C_0805" H 6325 3125 50  0001 C CNN
+F 3 "" H 6325 3275 50  0000 C CNN
+	1    6325 3275
+	1    0    0    -1
+$EndComp
+$Comp
+L +5V #PWR049
+U 1 1 5A24E07A
+P 6325 3100
+F 0 "#PWR049" H 6325 2950 50  0001 C CNN
+F 1 "+5V" H 6325 3240 50  0000 C CNN
+F 2 "" H 6325 3100 50  0000 C CNN
+F 3 "" H 6325 3100 50  0000 C CNN
+	1    6325 3100
+	1    0    0    -1
+$EndComp
+$Comp
+L GND #PWR050
+U 1 1 5A24E130
+P 6325 3450
+F 0 "#PWR050" H 6325 3200 50  0001 C CNN
+F 1 "GND" H 6325 3300 50  0000 C CNN
+F 2 "" H 6325 3450 50  0000 C CNN
+F 3 "" H 6325 3450 50  0000 C CNN
+	1    6325 3450
+	1    0    0    -1
+$EndComp
+Wire Wire Line
+	6325 3375 6325 3450
+Wire Wire Line
+	6325 3175 6325 3100
+NoConn ~ 5000 1800
+NoConn ~ 1300 2600
+$Comp
+L STM8S105K4 U2
+U 1 1 5A252F62
+P 3150 2500
+F 0 "U2" H 1950 3500 60  0000 C CNN
+F 1 "STM8S105K4" H 4050 3500 60  0000 C CNN
+F 2 "Housings_QFP:LQFP-32_7x7mm_Pitch0.8mm" H 3200 1200 60  0001 C CNN
+F 3 "http://www.st.com/st-web-ui/static/active/en/resource/technical/document/datasheet/CD00200092.pdf" H 3100 1350 60  0001 C CNN
+	1    3150 2500
+	1    0    0    -1
+$EndComp
+Wire Wire Line
+	1100 6050 1100 6100
+$Comp
+L AMS1117 U7
+U 1 1 5A25366F
+P 1250 7050
+F 0 "U7" H 1400 6854 50  0000 C CNN
+F 1 "AMS1117" H 1250 7250 50  0000 C CNN
+F 2 "TO_SOT_Packages_SMD:SOT-223" H 1300 6650 50  0001 C CNN
+F 3 "http://www.advanced-monolithic.com/pdf/ds1117.pdf" H 1400 6750 50  0001 C CNN
+	1    1250 7050
+	1    0    0    -1
+$EndComp
+Wire Wire Line
+	800  7000 850  7000
+Wire Wire Line
+	1250 7300 1250 7400
 $EndSCHEMATC
